File: PowerRail.sch (KiCad schematic (older format))
At the start: 0 parts

Commit message: Latest work
Changed lines of the file:
@@
 $Descr A4 11693 8268
 encoding utf-8
-Sheet 1 3
+Sheet 1 4
 Title "ADP5071 PowerRail"
 Date "2015-09-17"
@@
 F1 "ADP5071.sch" 60
 $EndSheet
+$Sheet
+S 3900 2950 1450 150
+U 563B4316
+F0 "TPS65530" 60
+F1 "TPS65530.sch" 60
+$EndSheet
 $EndSCHEMATC
