File: PowerRail.kicad_pcb (KiCad board)
At the start: 2 copper layers, 31.2 x 65.9 mm, 65 parts, among them P1 CONN_01X03, P2 CONN_01X03, P3 CONN_01X02, P4 CONN_01X02, P5 CONN_01X02, P6 CONN_01X02, P7 PIN, P8 POUT, T1 NET-TIE, U1 LT3472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

Commit message: latest at work
Parts:
- moved P1 45.3 mm to (127.3, 84.7), turned to 180 degrees
- moved C1 41.9 mm to (120.8, 87.2), turned to 180 degrees
- moved L1 38.4 mm to (121.5, 84.8), turned to 180 degrees
- moved C2 36.8 mm to (115.2, 86.4), turned to 0 degrees
- moved P2 34.7 mm to (105.7, 84.7), turned to 180 degrees
- moved L2 33.8 mm to (123.8, 80.0), turned to 90 degrees
- moved C4 33.1 mm to (109.1, 84.7), turned to 180 degrees
- moved R1 31.1 mm to (113.2, 83.8), turned to 270 degrees
- moved C3 31.1 mm to (111.4, 83.9), turned to 270 degrees
- moved C6 29.7 mm to (120.1, 80.5), turned to 0 degrees
- moved U1 29.3 mm to (116.4, 82.2), turned to 180 degrees
- moved P6 28.1 mm to (87.8, 85.2), turned to 270 degrees
- moved L5 27.4 mm to (87.2, 104.1), turned to 270 degrees
- moved C5 27.1 mm to (109.0, 81.7), turned to 180 degrees
- moved P5 25.9 mm to (85.2, 77.6), turned to 0 degrees
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Connections:
- net Net-(C6-Pad1) renamed /Extras/DN
Routing:
- added copper zone on F.Cu, net /Extras/+12V
- added copper zone on F.Cu, net /Extras/-7V
- added copper zone on F.Cu, net /Extras/DN
- added copper zone on F.Cu, net /Extras/FB
- added copper zone on F.Cu, net /Extras/FB+
- added copper zone on F.Cu, net /Extras/FB-
- added copper zone on F.Cu, net /Extras/SW+
- added copper zone on F.Cu, net /Extras/SW-
- added copper zone on F.Cu, net /Extras/SW3
- added copper zone on F.Cu, net /Extras/SW4
- added copper zone on F.Cu, net /Extras/VIN
- added copper zone on F.Cu, net /Extras/VIN_2V7_14V0
- added copper zone on F.Cu, net /Extras/VIN_2V7_5V5
- added copper zone on F.Cu, net /Extras/VOUT_12V
- added copper zone on F.Cu, net /Extras/VOUT_3V3
- removed copper zone on F.Cu, net /Additional/+12V
- removed copper zone on F.Cu, net /Additional/-7V
- removed copper zone on F.Cu, net /Additional/FB
- removed copper zone on F.Cu, net /Additional/FB+
- removed copper zone on F.Cu, net /Additional/FB-
- removed copper zone on F.Cu, net /Additional/SW+
- removed copper zone on F.Cu, net /Additional/SW-
- removed copper zone on F.Cu, net /Additional/SW3
- removed copper zone on F.Cu, net /Additional/SW4
- removed copper zone on F.Cu, net /Additional/VIN
- removed copper zone on F.Cu, net /Additional/VIN_2V7_14V0
- removed copper zone on F.Cu, net /Additional/VIN_2V7_5V5
- removed copper zone on F.Cu, net /Additional/VOUT_12V
- removed copper zone on F.Cu, net /Additional/VOUT_3V3
- removed copper zone on F.Cu, net Net-(C13-Pad1)
Other:
- board size 31.2 x 65.9 mm -> 47 x 38.4 mm
