File: PowerRail.kicad_pcb (KiCad board)
At the start: 2 copper layers, 125 x 92.4 mm, 127 parts, among them P1 CONN_01X03, P10 LEDS, P11 CONN_01X06, P12 CONN_01X02, P13 USB_OTG, P14 CONN_01X06, P15 JTI-PWR, P2 CONN_01X03, P3 CONN_01X02, P4 CONN_01X02, P5 CONN_01X02, P6 CONN_01X02, P7 PIN, P8 POUT, P9 ADJ, T1 NET-TIE, T2 NET-TIE, U1 LT3472, U2 LMR62014, U3 LM3674, U4 ADP5071, U5 TPS65530, U6 VEC2616

Commit message: Latest power stuff
Parts:
- P7: footprint Pin_Headers:Pin_Header_Angled_1x02 -> Pin_Headers:Pin_Header_Straight_1x02
- P8: footprint Pin_Headers:Pin_Header_Angled_1x03 -> Pin_Headers:Pin_Header_Straight_1x03
- R24: value 500k -> 453k
- R26: value 100k -> 150k
- T2: moved to B.Cu
- moved T2 29.9 mm to (194.4, 49.1)
- moved P15 22.1 mm to (176.2, 35.6), turned to 90 degrees
- moved P12 20.4 mm to (192.6, 27.5)
- moved P10 18.4 mm to (209.2, 27.5), turned to 0 degrees
- moved C45 8.24 mm to (194.6, 32.4), turned to 270 degrees
- moved C32 7.63 mm to (184.4, 33.7), turned to 0 degrees
- moved C33 7.09 mm to (205.2, 30.6), turned to 0 degrees
- moved P11 6.06 mm to (194.0, 61.3)
- moved C27 5.81 mm to (198.1, 28.1), turned to 0 degrees
- moved R15 4.21 mm to (195.6, 38.6), turned to 0 degrees
- moved P14 4.10 mm to (176.2, 46.4)
- moved P9 3.62 mm to (214.3, 41.8)
- moved P13 3.45 mm to (180.3, 26.8)
- moved L13 3.23 mm to (190.6, 32.4), turned to 180 degrees
- moved D4 2.82 mm to (198.1, 36.8)
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Connections:
- net /TPS65530/V_BADJ renamed /TPS65530/B-ADJ
- net Net-(C30-Pad1) renamed /TPS65530/FB6
- net Net-(C33-Pad1) renamed /TPS65530/SWOUT
- net Net-(C36-Pad2) renamed /TPS65530/SS
- net Net-(C38-Pad2) renamed /TPS65530/REF
- net Net-(D4-Pad2) renamed /TPS65530/SW5
- net Net-(D5-Pad2) renamed /TPS65530/SW7
- net Net-(D6-Pad1) renamed /TPS65530/SW6
- net Net-(L10-Pad2) renamed /TPS65530/LL8
- net Net-(L15-Pad1) renamed /TPS65530/SW1
- net Net-(L17-Pad1) renamed /TPS65530/SW2S
- net Net-(L17-Pad2) renamed /TPS65530/SW2I
- net Net-(P10-Pad2) renamed /TPS65530/CIN
- net Net-(P9-Pad1) renamed /TPS65530/ADJ
- net Net-(R16-Pad2) renamed /TPS65530/S56
- net Net-(R19-Pad1) renamed /TPS65530/FB8
- net Net-(R20-Pad1) renamed /TPS65530/FBC
- net Net-(R24-Pad2) renamed /TPS65530/FBV
- net Net-(R29-Pad2) renamed /TPS65530/FB4
- net Net-(R31-Pad2) renamed /TPS65530/FB2
- net Net-(U5-Pad26) renamed /TPS65530/SW8LD
- net Net-(U5-Pad28) renamed /TPS65530/SW8HD
- C41 pad 1: /TPS65530/VCC1 -> /TPS65530/VBATT
- C42 pad 1: /TPS65530/VCC3 -> /TPS65530/VBATT
- C43 pad 1: /TPS65530/VCC2 -> /TPS65530/VBATT
- C44 pad 1: /TPS65530/VCC4 -> /TPS65530/VBATT
- C45 pad 2: /TPS65530/VCC6 -> /TPS65530/VBATT
- C46 pad 1: /TPS65530/VCC8 -> /TPS65530/VBATT
- C47 pad 1: /TPS65530/VCC8 -> /TPS65530/VBATT
- C48 pad 2: /TPS65530/VCC7 -> /TPS65530/VBATT
- L10 pad 1: /TPS65530/VCC8 -> /TPS65530/VBATT
- L11 pad 1: /TPS65530/VCC7 -> /TPS65530/VBATT
- U5 pad 12: /TPS65530/VCC2 -> /TPS65530/VBATT
- U5 pad 18: /TPS65530/VCC1 -> /TPS65530/VBATT
- U5 pad 23: /TPS65530/VCC3 -> /TPS65530/VBATT
- U5 pad 40: /TPS65530/VCC5 -> /TPS65530/VBATT
- U5 pad 42: /TPS65530/VCC6 -> /TPS65530/VBATT
- U5 pad 48: /TPS65530/VCC4 -> /TPS65530/VBATT
Routing:
- net /TPS65530/VBATT: track 0.00 -> 246.4 mm, vias 0 -> 9
- net GNDPWR: track 12.5 -> 114.1 mm, vias 0 -> 28
- net GND: track 64.1 -> 117.9 mm, vias 23 -> 31
- net /TPS65530/VOUT_MOTOR_5V: track 0.00 -> 52.1 mm
- net /TPS65530/CIN: track 0.00 -> 33.3 mm
- net /TPS65530/VOUT_AFE_3V3: track 16.1 -> 43.8 mm
- net /TPS65530/VOUT_MEM_1V8: track 0.00 -> 27.0 mm
- net /TPS65530/VOUT_BACKL_5V: track 0.00 -> 26.2 mm
- net /TPS65530/SW8LD: track 0.00 -> 23.0 mm
- net /TPS65530/SWOUT: track 0.00 -> 18.7 mm
- net /TPS65530/EN_LGT: track 0.00 -> 18.0 mm, vias 0 -> 2
- net /TPS65530/XSLEEP: track 0.00 -> 17.7 mm, vias 0 -> 2
- net /TPS65530/EN_AFE: track 0.00 -> 17.7 mm, vias 0 -> 2
- net /TPS65530/B-ADJ: track 0.00 -> 16.1 mm, vias 0 -> 2
- net /TPS65530/SW7: track 0.00 -> 16.1 mm
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- added copper zone on F.Cu, net /Extras/+12V
- added copper zone on F.Cu, net /Extras/-7V
- added copper zone on F.Cu, net /Extras/FB
- added copper zone on F.Cu, net /Extras/FB+
- added copper zone on F.Cu, net /Extras/FB-
- added copper zone on F.Cu, net /Extras/SW-
- added copper zone on F.Cu, net /Extras/SW3
- added copper zone on F.Cu, net /Extras/SW4
- added copper zone on F.Cu, net /Extras/VIN
- added copper zone on F.Cu, net /Extras/VIN_2V7_14V0
- added copper zone on F.Cu, net /Extras/VIN_2V7_5V5
- added copper zone on F.Cu, net /Extras/VOUT_12V
- added copper zone on F.Cu, net /Extras/VOUT_3V3
- added copper zone on F.Cu, net /TPS65530/VBATT
- added copper zone on B.Cu, net GNDPWR
- added copper zone on F.Cu, net GNDPWR
- removed copper zone on F.Cu, net /Additional/+12V
- removed copper zone on F.Cu, net /Additional/-7V
- removed copper zone on F.Cu, net /Additional/FB
- removed copper zone on F.Cu, net /Additional/FB+
- removed copper zone on F.Cu, net /Additional/FB-
- removed copper zone on F.Cu, net /Additional/SW-
- removed copper zone on F.Cu, net /Additional/SW3
- removed copper zone on F.Cu, net /Additional/SW4
- removed copper zone on F.Cu, net /Additional/VIN
- removed copper zone on F.Cu, net /Additional/VIN_2V7_14V0
- removed copper zone on F.Cu, net /Additional/VIN_2V7_5V5
- removed copper zone on F.Cu, net /Additional/VOUT_12V
- removed copper zone on F.Cu, net /Additional/VOUT_3V3
Other:
- board size 125 x 92.4 mm -> 122 x 91.4 mm
- rule trace_min: 0.1524 -> 0.127

Commit message: Latest work
Parts:
- removed C1, C2, C8, C9: 2.2uF, Capacitors_SMD:C_0603
- removed C10: 4.7uF, smd:SM0603
- removed C11: 6.8pF, smd:SM0603
- removed C12: 33pF, smd:SM0603
- removed C13: 10uF, smd:SM0603
- removed C14: 220pF, Capacitors_SMD:C_0603
- removed C15: 4.7uF, Capacitors_SMD:C_0603
- removed C16: 3.9nF, smd:SM0603
- removed C17: 22.0uF, smd:SM1206
- removed C18: 12pF, smd:SM0603
- removed C19: 8.2nF, smd:SM0603
- removed C20: 68pF, smd:SM0603
- removed C21, C22: 1.0uF, smd:SM0603
- removed C23: 4.7uF, smd:SM0805
- removed C24: 1.0uF, smd:SM0805
- removed C25, C26: 10.0uF, smd:SM1206
- removed C3: 4.7pF, Capacitors_SMD:C_0603
- removed C4, C5: 0.1uF, Capacitors_SMD:C_0603
- removed C6: 1.0uF, Capacitors_SMD:C_0603
- removed C7: 10pF, Capacitors_SMD:C_0603
- removed D1: D_Schottky, engstad:diode-smd-powerdi-123
- removed D2, D3: DFLS240, engstad:diode-smd-powerdi-123
- removed L1: 22uH, SMD_Packages:SMD-1210_Pol
- removed L2, L3: 47uH, SMD_Packages:SMD-1210_Pol
- removed L4: 10 uH, engstad:inductor-smd-1212
- removed L5: 2.2uH, SMD_Packages:SMD-1210_Pol
- removed L6: 2.2uH, engstad:inductor-smd-xal40
- removed L7: 3.3uH, SMD_Packages:SMD-1210_Pol
- removed L8: 0.47uH, SMD_Packages:SMD-1210_Pol
- removed L9: 1.0uH, SMD_Packages:SMD-1210_Pol
- removed P1, P2: CONN_01X03, Pin_Headers:Pin_Header_Straight_1x03
- removed P3, P4, P5, P6: CONN_01X02, Pin_Headers:Pin_Header_Straight_1x02
- removed P7: PIN, Pin_Headers:Pin_Header_Straight_1x02
- removed P8: POUT, Pin_Headers:Pin_Header_Straight_1x03
- removed R1: 430k, Resistors_SMD:R_0603
- removed R10: 6.98k, smd:SM0603
- removed R11: 66.5k, smd:SM0603
- removed R12: 68.1k, smd:SM0603
- removed R13: 3.09 Ohm, smd:SM0603
- removed R14: 6.19 Ohm, smd:SM0603
- removed R2: 280k, Resistors_SMD:R_0603
- removed R3: 562k, smd:SM0603
- removed R4: 100k, smd:SM0603
- removed R5: 117k, Resistors_SMD:R_0603
- removed R6: 13.3k, Resistors_SMD:R_0603
- removed R7: 21.5k, smd:SM0603
- removed R8: 5.23k, smd:SM0603
- removed R9: 4.75k, smd:SM0603
- removed T1, T2: NET-TIE, Oddities:NetTie-I_Connected_SMD
- removed U1: LT3472, Housings_DFN_QFN:DFN-10-1EP_3x3mm_Pitch0.5mm
- removed U2: LMR62014, Housings_SOT-23_SOT-143_TSOT-6:SOT-23-5
- removed U3: LM3674, Housings_SOT-23_SOT-143_TSOT-6:SOT-23-5
- removed U4: ADP5071, Housings_DFN_QFN:QFN-20-1EP_4x4mm_Pitch0.5mm
- added hole_3mm: VAL**, w_details:hole_3mm, F.Cu at (148.9, 74.0)
- added hole_3mm: VAL**, w_details:hole_3mm, F.Cu at (172.4, 75.3)
- added hole_3mm: VAL**, w_details:hole_3mm, F.Cu at (172.4, 110.9)
- added hole_3mm: VAL**, w_details:hole_3mm, F.Cu at (136.8, 110.9)
- moved P14 67.9 mm to (135.5, 100.7)
- moved P10 66.2 mm to (171.1, 81.7), turned to 270 degrees
- moved P15 64.4 mm to (135.5, 85.6)
- moved P11 64.3 mm to (154.6, 112.1)
- moved R18 64.3 mm to (154.9, 89.8)
- moved R15 64.2 mm to (154.9, 88.3)
- moved C36 64.0 mm to (146.4, 95.4)
- moved C49 64.0 mm to (171.2, 96.6)
- moved D5 64.0 mm to (165.1, 89.1)
- moved D6 64.0 mm to (148.7, 87.6)
- moved L12 64.0 mm to (160.6, 82.4)
- moved L13 64.0 mm to (150.6, 82.4)
- moved R16 64.0 mm to (151.5, 89.9), turned to 0 degrees
- moved R21 64.0 mm to (171.2, 95.1)
- moved R25 64.0 mm to (159.4, 94.9)
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Connections:
- C30 pad 1: /TPS65530/FB6 -> GND
- C30 pad 2: GND -> /TPS65530/S56
- R16 pad 1: /TPS65530/FB6 -> /TPS65530/VOUT_CCD-
- R16 pad 2: /TPS65530/S56 -> /TPS65530/FB6
- R17 pad 1: /TPS65530/VOUT_CCD- -> /TPS65530/S56
Routing:
- net /TPS65530/VBATT: track 246.4 -> 160.5 mm
- net GND: track 117.9 -> 50.8 mm, vias 31 -> 7
- net GNDPWR: track 114.1 -> 52.5 mm, vias 28 -> 32
- net +5V: track 27.7 -> 0.00 mm, vias 2 -> 0
- net /ADP5071/0V: track 21.9 -> 0.00 mm, vias 1 -> 0
- net /Extras/FB2: track 17.8 -> 0.00 mm, vias 2 -> 0
- net /ADP5071/12V0: track 16.7 -> 0.00 mm
- net /TPS65530/SW8LD: track 23.0 -> 7.60 mm, vias 0 -> 2
- net /ADP5071/-7V0: track 14.9 -> 0.00 mm, vias 2 -> 0
- net /TPS65530/CIN: track 33.3 -> 21.3 mm, vias 0 -> 1
- net /ADP5071/+12V: track 12.0 -> 0.00 mm
- net /Extras/~SHDN: track 11.1 -> 0.00 mm
- net /Extras/VIN: track 10.2 -> 0.00 mm
- net /ADP5071/SW1: track 8.78 -> 0.00 mm
- net /ADP5071/-7V: track 8.56 -> 0.00 mm
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- added copper zone on F.Cu, net /TPS65530/VOUT_MOTOR_5V
- added copper zone on In2.Cu, net GND
- added copper zone on In1.Cu, net GNDPWR
- removed copper zone on F.Cu, net +5V
- removed copper zone on F.Cu, net /ADP5071/+12V
- removed copper zone on F.Cu, net /ADP5071/-7V
- removed copper zone on F.Cu, net /ADP5071/-7V0
- removed copper zone on F.Cu, net /ADP5071/0V
- removed copper zone on F.Cu, net /ADP5071/12V0
- removed copper zone on F.Cu, net /ADP5071/INBK
- removed copper zone on F.Cu, net /ADP5071/SW1
- removed copper zone on F.Cu, net /ADP5071/SW2
- removed copper zone on F.Cu, net /Additional/SW+
- removed copper zone on F.Cu, net /Extras/+12V
- removed copper zone on F.Cu, net /Extras/-7V
- removed copper zone on F.Cu, net /Extras/FB
- removed copper zone on F.Cu, net /Extras/FB+
- removed copper zone on F.Cu, net /Extras/FB-
- removed copper zone on F.Cu, net /Extras/SW-
- removed copper zone on F.Cu, net /Extras/SW3
- removed copper zone on F.Cu, net /Extras/SW4
- removed copper zone on F.Cu, net /Extras/VIN
- removed copper zone on F.Cu, net /Extras/VIN_2V7_14V0
- removed copper zone on F.Cu, net /Extras/VIN_2V7_5V5
- removed copper zone on F.Cu, net /Extras/VOUT_12V
- removed copper zone on F.Cu, net /Extras/VOUT_3V3
- removed copper zone on B.Cu, net GNDPWR
- removed copper zone on F.Cu, net Net-(C13-Pad1)
Other:
- board size 122 x 91.4 mm -> 43.2 x 43.2 mm
- copper layers 2 -> 4
- net class Default: clearance 0.2 -> 0.05
- rule trace_clearance: 0.2 -> 0.05
- board text added: "+"
- board text added: "+12V"
- board text added: "-"
- board text added: "-7V"
- board text added: "0.0"
- board text added: "0V"
- board text added: "1.2"
- board text added: "1.8"
- board text added: "3.3"
- board text added: "5.0"
- board text added: "5Vin"
- board text added: "AFE"
- board text added: "CCD"
- board text added: "LGT"
- board text added: "SEQ"
- board text added: "~SLP~"
- board text removed: "Vin 2.7-5.5V"
- board text removed: "Vout 3.3V"
