File: extras.sch (KiCad schematic (older format))
At the start: 36 parts, among them P1 CONN_01X03, P2 CONN_01X03, P3 CONN_01X02, P4 CONN_01X02, P5 CONN_01X02, P6 CONN_01X02, U1 LT3472, U2 LMR62014, U3 LM3674

Commit message: latest at work
Connections:
- net labels added: DN
Changed lines of the file:
@@
 EESchema Schematic File Version 2
-LIBS:PowerRail-rescue
 LIBS:power
 LIBS:device
@@
 LIBS:xess
 LIBS:xilinx7
-LIBS:engstad
 LIBS:PowerRail-cache
 EELAYER 25 0
@@
 Text Label 9300 1800 0    60   ~ 0
 SW3
+Text Label 3800 1800 0    60   ~ 0
+DN
 $EndSCHEMATC
