File: TPS65530.sch (KiCad schematic (older format))
At the start: 62 parts, among them P10 LEDS, P11 CONN_01X06, P12 CONN_01X02, P13 USB_OTG, P14 CONN_01X06, P15 JTI-PWR, P9 ADJ, T2 NET-TIE, U5 TPS65530, U6 VEC2616

Commit message: Latest power stuff
Parts:
- R24: value 500k -> 453k
- R26: value 100k -> 150k
Connections:
- net VCC1 is gone; now on net VBATT: C41.1, U5.18 (VCC1)
- net VCC2 is gone; now on net VBATT: C43.1, U5.12 (VCC2)
- net VCC3 is gone; now on net VBATT: C42.1, U5.23 (VCC3)
- net VCC4 is gone; now on net VBATT: C44.1, U5.48 (VCC4)
- net VCC5 is gone; now on net VBATT: U5.40 (VCC5)
- net VCC6 is gone; now on net VBATT: C45.2, U5.42 (VCC6)
- net VCC7 is gone; now on net VBATT: C48.2, L11.1
- net VCC8 is gone; now on net VBATT: C46.1, C47.1, L10.1
- net REF: now reaches C38.2, U5.11 (REF)
- net SW2S: now reaches L17.1, U5.13 (SW2S)
- net SW2I: now reaches L17.2, U5.15 (SW2I)
- net FB2: now reaches R31.2, R32.1, U5.17 (FB2)
- net SW1: now reaches L15.1, U5.19 (SW1)
- net SW8LD: now reaches U5.26 (SW8LD), U6.2
- net LL8: now reaches L10.2, U5.27 (LL8), U6.5, U6.6, U6.7, U6.8
- net SW8HD: now reaches U5.28 (SW8HD), U6.4
- net FB8: now reaches R19.1, R25.2, U5.30 (FB8)
- net FBC: now reaches R20.1, U5.33 (FBC)
- net CIN: now reaches P10.2 (P2), U5.34 (CIN)
- net FBV: now reaches R24.2, R26.2, U5.35 (FBV)
- net SW7: now reaches D5.2 (A), L11.2, U5.36 (SW7)
- net SW5: now reaches D4.2 (A), L12.2, U5.38 (SW5)
- net SWOUT: now reaches C33.1, L12.1, U5.39 (SWOUT)
- net SW6: now reaches D6.1 (K), L13.1, U5.43 (SW6)
- net FB6: now reaches C30.1, R16.1, R17.2, U5.44 (FB6)
- net S56: now reaches R16.2, U5.45 (S/S56)
- net FB4: now reaches R29.2, R30.1, U5.5 (FB4)
- net SS: now reaches C36.2, U5.9 (S/S)
- net ADJ: now reaches P9.1 (P1), R21.2
- net V_BADJ renamed B-ADJ
Other:
- moved on the sheet: C36, C38, L15, P9, R24, R26, R33, R34

Commit message: Latest work
Connections:
- net FB6: now also R16.2; no longer C30.1, R16.1
- net GND: now also C30.1; no longer C30.2
- net S56: now also C30.2, R17.1; no longer R16.2
- net VOUT_CCD-: now also R16.1; no longer R17.1
Other:
- note added: "R1"
- note added: "R2"
- moved on the sheet: C30, R17

Commit message: More work
Parts:
- D4, D5, D6: footprint Diodes_SMD:SOD-123 -> engstad:diode-sod-123
- P13: footprint w_conn_pc:conn_usb_B_mini_smd -> engstad:conn-smd-usb-b-mini
- P15: footprint xess:HDR_1x2 -> w_conn_jst-ph:b2b-ph-kl
- T2: footprint Oddities:NetTie-I_Connected_SMD -> engstad:net-tie-0.5mm
- U5: footprint Housings_DFN_QFN:UQFN-48-1EP_6x6mm_Pitch0.4mm -> engstad:qfn-48-p
Connections:
- net GND: now also P15.1 (P1); no longer P15.2 (P2)
- net VBATT: now also P15.2 (P2); no longer P15.1 (P1)

Commit message: Fixes
Parts:
- L17: footprint engstad:inductor-smd-50x50 -> engstad:inductor-smd-2020-50x50
Changed lines of the file:
@@
 F 0 "L17" H 4980 4440 50  0000 L CNN
 F 1 "3.3uH/3.3A" H 4980 4360 50  0000 L CNN
-F 2 "engstad:inductor-smd-50x50" H 4950 4400 60  0001 C CNN
+F 2 "engstad:inductor-smd-2020-50x50" H 4950 4400 60  0001 C CNN
 F 3 "" H 4950 4400 60  0000 C CNN
 F 4 "Murata" H 4950 4400 60  0001 C CNN "Manufacturer"

Commit message: Tiny fixes
Other:
- moved on the sheet: C27, C48, L17

Commit message: Safety checkin.
Parts:
- removed T2: NET-TIE, engstad:net-tie-0.5mm, symbol NET-TIE
- removed U6: VEC2616, engstad:sot-28fl, symbol VEC2616
- added NT1: Net-Tie_2, symbol Device:Net-Tie_2
- added NT?: Net-Tie_3_Tee, symbol Device:Net-Tie_3_Tee
- added Q1: VEC2616, symbol Engstad:VEC2616
- added R37, R38, R39: 10, smd:SM0603, symbol Device:R
- added T10, T11, T12, T13, T14, T15, T3, T4, T5, T6, T7, T8, T9: NET-TIE, engstad:net-tie-0.5mm, symbol Device:Net-Tie_2
- added U6: AP2161W, Package_TO_SOT_SMD:SOT-23-5, symbol Power_Management:AP2161W
- C27, C29, C30, C32, C33, C34, C35, C36, C37, C38, C39, C40, C41, C42, C43, C44, C45, C46, C47, C48: symbol C_Small -> Device:C_Small
- C28, C31: symbol C -> Device:C_Small
- C49: value C_Small -> 0.1uF; symbol C_Small -> Device:C_Small
- D4, D5, D6: symbol D_Small -> Device:D_Small
- L10, L12, L13: symbol L_Small -> Device:L
- L11: symbol INDUCTOR -> Device:L
- L14, L15, L16, L17: symbol L_Small -> Device:L_Small
- P10, P12, P15: symbol CONN_01X02 -> Connector_Generic:Conn_01x02
- P11, P14: symbol CONN_01X06 -> Connector_Generic:Conn_01x06
- P13: symbol USB_OTG -> Connector:USB_OTG
- P9: symbol CONN_01X01 -> Connector_Generic:Conn_01x01
- R15, R16, R17, R18, R27, R28, R29, R30, R31, R32, R33, R34: symbol R_Small -> Device:R_Small
- R19, R20, R21, R24, R25, R26: symbol R -> Device:R
- U5: symbol TPS65530 -> Engstad:TPS65530
Connections:
- net FB1: now also R34.1; no longer R34.2
- net FB3: now also R27.1, R28.2; no longer R27.2, R28.1
- net FB6: now also R16.1, R17.1; no longer R16.2, R17.2
- net FB8: now also R19.2, R25.1; no longer R19.1, R25.2
- net FBG78: now also R25.2; no longer R25.1
- net GND: now also NT?.3; no longer C30.1, C36.1, C38.1, C49.2, P13.6 (shield), P14.6 (P6), R18.2, R28.2, R30.2, R32.2, R34.1, U5.10 (AGND)
- net GNDPWR: now also NT1.2, NT?.2, T11.2, T12.2, T13.2, T14.2, T15.1; no longer C27.2, C28.2, C29.2, C31.2, C32.1, C33.2, C34.2, C35.1, C37.2, C39.2, C40.2, C41.2, C42.2, C43.2, C44.2, C45.1, C46.2, C47.2, C48.1, L13.2, R20.2, U5.14 (PGND2), U5.2 (PGND4), U5.20 (PGND1), U5.25 (PGND3), U5.37 (PGND5/7)
- net LL8: now also R38.2; no longer L10.2
- net REF: now also C38.1; no longer C38.2
- net SS: now also C36.1; no longer C36.2
- net SW5: now also L12.1; no longer L12.2
- net SW6: now also L13.2; no longer L13.1
- net SWOUT: now also L12.2; no longer L12.1
- net VOUT_CCD+: now also R15.1; no longer R15.2
- net VOUT_CCD-: now also R16.2; no longer R16.1
- net VOUT_MEM_1V8: now also R27.2; no longer R27.1
- net SW3: now reaches L14.1, U5.24 (SW3)
- net FB5: now reaches R18.1, U5.41 (FB5)
- net FB5: now also R15.2; no longer R15.1
- net CIN renamed VDD_LED
- net EN_SEQ renamed SEQ56_CTL
- net SEQ56_CTL: no longer U5.47 (SEQ56)
- removed net S56: C30.2, R17.1, U5.45 (S/S56)
- net SW8HD renamed SW8H
- net SW8H: now also R37.1
- net SW8LD renamed SW8L
- net SW8L: now also R39.1
- removed net VBATT: C41.1, C42.1, C43.1, C44.1, C45.2, C46.1, C47.1, C48.2, L10.1, L11.1, P13.1 (VCC), P15.2 (P2), U5.12 (VCC2), U5.18 (VCC1), U5.23 (VCC3), U5.40 (VCC5), U5.42 (VCC6), U5.48 (VCC4)
- net VOUT_BACKL_5V renamed VCC_LED
- net VOUT_MOTOR_5V renamed VOUT_5V
- net VOUT_5V: now also R19.1, Q1.3 (S); no longer R19.2
- new net: C27.2, C29.2, C32.1, C33.2, C45.2, C48.2, C49.2, L13.1, R18.2, R20.2, T15.2, U5.37 (PGND5/7)
- new net: L10.2, Q1.5, Q1.6 (D), Q1.7, Q1.8 (D), R38.1
- new net: Q1.2 (G), R39.2
- new net: Q1.4 (G), R37.2
- new net GNDA: C30.2, C36.2, C38.2, NT?.1, P14.6 (Pin_6), U5.10 (AGND)
- new net PGND1: C37.2, C41.2, R34.2, T11.1, U5.20 (PGND1)
- new net PGND2: C40.2, C43.2, R32.2, T14.1, U5.14 (PGND2)
- new net PGND3: C35.1, C42.2, R28.1, T12.1, U5.25 (PGND3)
- new net PGND4: C39.2, C44.2, R30.2, T13.1, U5.2 (PGND4)
- new net PGND8: C28.2, C31.2, C34.2, C46.2, C47.2, NT1.1, Q1.1 (S)
- new net SEQ56_CTRL: U5.47 (SEQ56)
- new net SS56: C30.1, R17.2, U5.45 (S/S56)
- new net VBUS: P13.1 (VBUS), P15.2 (Pin_2), T10.2, T3.2, T4.2, T5.2, T6.2, T7.2, T8.2, T9.2
- new net VCC1: C41.1, T3.1, U5.18 (VCC1)
- new net VCC2: C43.1, T4.1, U5.12 (VCC2)
- new net VCC3: C42.1, T5.1, U5.23 (VCC3)
- new net VCC4: C44.1, T6.1, U5.48 (VCC4)
- new net VCC5: T7.1, U5.40 (VCC5)
- new net VCC6: C45.1, T8.1, U5.42 (VCC6)
- new net VCC7: C48.1, L11.1, T9.1
- new net VCC8: C46.1, C47.1, L10.1, T10.1
- no-connect marks 3 -> 4
Other:
- note added: "If VBUS < 2.5 V, then instead, VCC1, VCC3 and \nVCC6 should be connected to channel 8 output."
- note added: "PS (Power Source): Power input for IC"
- note added: "VOUT=1.25-(1+R2/R1)*1.25 [V]"
- note removed: "-1.35[A]"
- note removed: "PS: Power input for IC"
- note removed: "VOUT=\n1.25-(1+R2/R1)*1.25 [V]"
- moved on the sheet: C27, C28, C29, C30, C31, C32, C33, C34, C35, C36, C37, C38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
